File: PCB_Files/65MX.kicad_pcb (KiCad board)
At the start: 2 copper layers, 303.8 x 94.2 mm, 135 parts, among them J1 jst_sh, SW1 NRST, SW2 NRST, U1 STM32F072CBTx, U2 SRV05-4, U3 XC6206PxxxMR

Commit message: made a readme
Routing:
- net +3V3: track 63.7 -> 55.2 mm
- net Net-(D31-A2): track 59.5 -> 61.4 mm
- net D+: track 30.0 -> 31.4 mm
- net COL2: track 176.1 -> 175.5 mm
- net GND: track 44.7 -> 44.6 mm, vias 79 -> 81

Commit message: Boot+Reset silkscreen
added a silkscreen next to the boot and reset switches to differentiate between then
Other:
- board text added: "boot"
- board text added: "reset"

Commit message: moved plate holes
moved plate holes to enable proper gummy o ring mounting
Parts:
- moved H3 28.0 mm to (104.4, 165.1)
- moved H1 19.4 mm to (98.4, 98.4)
- moved H2 11.4 mm to (365.1, 98.4)
- moved C8 9.80 mm to (102.8, 107.6), turned to 0 degrees
- moved D34 9.13 mm to (365.1, 149.6)
- moved H4 7.94 mm to (365.1, 155.6)
- moved U3 5.98 mm to (102.8, 104.4), turned to 180 degrees
- moved D33 4.76 mm to (346.1, 154.0)
- moved C7 3.94 mm to (102.8, 101.2), turned to 0 degrees
Routing:
- net +3V3: track 55.2 -> 42.4 mm
- net Net-(D34-A2): track 73.0 -> 61.7 mm
- net COL6: track 242.4 -> 235.3 mm
- net GND: track 44.6 -> 37.8 mm, vias 81 -> 84
- net +5V: track 26.8 -> 32.7 mm
- net COL5: track 187.3 -> 181.6 mm
- net COL13: track 333.4 -> 329.7 mm
- net Net-(D34-A1): track 11.2 -> 14.9 mm
- net COL11: track 283.8 -> 280.8 mm
- net COL8: track 204.6 -> 201.6 mm
- net COL3: track 175.4 -> 172.3 mm
- net COL10: track 264.4 -> 261.3 mm
- net COL1: track 95.2 -> 92.2 mm
- net COL4: track 198.9 -> 195.9 mm
- net COL2: track 175.5 -> 172.5 mm
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